File: Hardware/Electrical/gp-shield/_autosave-power.kicad_sch (KiCad schematic)
At the start: 30 parts, among them J1 XT60/TERM2, J2 XT60/TERM2, Q1 Q_PMOS_GDS, SW1 SW_SPDT, U1 NCP1117-5.0_SOT223, U2 LM4040DBZ-2.5, U4 LM397

Commit message: Major revisions
Parts:
- C5: footprint Capacitor_SMD:CP_Elec_8x5.4 -> Capacitor_THT:CP_Radial_D8.0mm_P3.50mm
Changed lines of the file:
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@@
       (effects (font (size 1.27 1.27)) (justify left))
     )
-    (property "Footprint" "Capacitor_SMD:CP_Elec_8x5.4" (id 2) (at 213.0552 48.26 0)
+    (property "Footprint" "Capacitor_THT:CP_Radial_D8.0mm_P3.50mm" (id 2) (at 213.0552 48.26 0)
       (effects (font (size 1.27 1.27)) hide)
     )
